File: pcb-project/pcb-project.sch (KiCad schematic (older format))
At the start: 24 parts, among them SW1 SW_Push, U1 ATmega32U4-A, Y1 16MHz

Commit message: PCB Routing
Parts:
- renumbered MX3 to MX2, MX2 to MX3
Changed lines of the file:
@@
 	6600 3550 6500 3550
 $Comp
-L MX_Alps_Hybrid:MX-NoLED MX3
+L MX_Alps_Hybrid:MX-NoLED MX2
 U 1 1 6098CC99
 P 7600 3400
-F 0 "MX3" H 7633 3623 60  0000 C CNN
+F 0 "MX2" H 7633 3623 60  0000 C CNN
 F 1 "MX-NoLED" H 7633 3549 20  0000 C CNN
 F 2 "MX_Alps_Hybrid:MX-1U-NoLED" H 6975 3375 60  0001 C CNN
@@
 	7550 3550 7450 3550
 $Comp
-L MX_Alps_Hybrid:MX-NoLED MX2
+L MX_Alps_Hybrid:MX-NoLED MX3
 U 1 1 60995455
 P 6650 4200
-F 0 "MX2" H 6683 4423 60  0000 C CNN
+F 0 "MX3" H 6683 4423 60  0000 C CNN
 F 1 "MX-NoLED" H 6683 4349 20  0000 C CNN
 F 2 "MX_Alps_Hybrid:MX-1U-NoLED" H 6025 4175 60  0001 C CNN
