File: rqm-pcb/rqm-pcb.sch (KiCad schematic (older format))
At the start: 24 parts, among them J1 USB_mini_micro_B, K1 KEYSW, K2 KEYSW, K3 KEYSW, K4 KEYSW, SW1 SW_PUSH, U1 ATMEGA32U4, X1 XTAL_GND

Commit message: RQM complete
Parts:
- C1, C2, C3, C4, C5, C6, C7, C8: footprint (none) -> Capacitor_SMD:C_0805_2012Metric_Pad1.18x1.45mm_HandSolder
- D1, D2, D3, D4: footprint (none) -> keyboard_parts:D_SOD123_axial
- J1: footprint (none) -> keyboard_parts:USB_miniB_hirose_5S8
- K1, K2, K3, K4: footprint (none) -> keebs:Mx_Alps_100
- R1: renamed from R?; footprint (none) -> Resistor_SMD:R_0805_2012Metric_Pad1.20x1.40mm_HandSolder
- R2, R3, R4: footprint (none) -> Resistor_SMD:R_0805_2012Metric_Pad1.20x1.40mm_HandSolder
- SW1: footprint (none) -> Button_Switch_SMD:SW_SPST_TL3342
- U1: footprint (none) -> Housings_QFP:TQFP-44_10x10mm_Pitch0.8mm
- X1: footprint (none) -> Crystal:Crystal_SMD_SeikoEpson_FA238-4Pin_3.2x2.5mm_HandSoldering
Connections:
- net VCC: now also U1.7 (VBus)
- no-connect marks 24 -> 23
Other:
- moved on the sheet: C1, C2, C3, C4, C5, C6, C7, C8, D1, D2, D3, D4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
